File: hard/XS40.sch (KiCad schematic (older format))
At the start: 94 parts, among them J1 USB_B_Micro, J2 Conn_01x20_Female, J3 Nu-link, SW1 SW_Push, SW10 SW_Push, SW11 SW_Push, SW12 SW_Push, SW13 SW_Push, SW14 SW_Push, SW15 SW_Push, SW16 SW_Push, SW17 SW_Push, SW18 SW_Push, SW19 SW_Push, SW2 SW_Push, SW20 SW_Push, SW21 SW_Push, SW22 SW_Push, SW23 SW_Push, SW24 SW_Push, SW25 SW_Push, SW26 SW_Push, SW27 SW_Push, SW28 SW_Push, SW29 SW_Push, SW3 SW_Push, SW30 SW_Push, SW31 SW_Push, SW32 SW_Push, SW33 SW_Push, SW34 SW_Push, SW35 SW_Push, SW36 SW_Push, SW37 SW_Push, SW38 SW_Push, SW39 SW_Push, SW4 SW_Push, SW40 SW_Push, SW5 SW_Push, SW6 SW_Push, SW7 SW_Push, SW8 SW_Push, SW9 SW_Push, U1 N76E003AT20, U2 CH9328

Commit message: 更新PCB图
Parts:
- J1: footprint Connector_USB:USB_Micro-B_GCT_USB3076-30-A -> Connector_USB:USB_Micro-B_Molex-105017-0001
- U1: symbol MCU_Nuvoton:N76E003AT20 -> XS40-rescue:N76E003AT20-MCU_Nuvoton
- U2: symbol ch9328:CH9328 -> XS40-rescue:CH9328-ch9328
Connections:
- net COL7: now also J3.4 (Pin_4); no longer J3.2 (Pin_2)
- net GND: now also J3.1 (Pin_1); no longer J3.5 (Pin_5)
- net RST: now also J3.2 (Pin_2); no longer J3.4 (Pin_4)
- net VDD: now also J3.5 (Pin_5); no longer J3.1 (Pin_1)
Other:
- moved on the sheet: J3
Changed lines of the file:
@@
 COL8
 $Comp
-L MCU_Nuvoton:N76E003AT20 U1
+L XS40-rescue:N76E003AT20-MCU_Nuvoton U1
 U 1 1 5E6CF047
 P 4100 5000
@@
 F 0 "J1" H 1607 7367 50  0000 C CNN
 F 1 "USB_B_Micro" H 1607 7276 50  0000 C CNN
-F 2 "Connector_USB:USB_Micro-B_GCT_USB3076-30-A" H 1700 6850 50  0001 C CNN
+F 2 "Connector_USB:USB_Micro-B_Molex-105017-0001" H 1700 6850 50  0001 C CNN
 F 3 "~" H 1700 6850 50  0001 C CNN
 	1    1550 6900
@@
 	1550 7350 1550 7300
 $Comp
-L ch9328:CH9328 U2
+L XS40-rescue:CH9328-ch9328 U2
 U 1 1 5E810AB5
 P 4900 6750
@@
 L Connector:Conn_01x05_Male J3
 U 1 1 5F0A293A
-P 900 5000
-F 0 "J3" H 1008 5381 50  0000 C CNN
-F 1 "Nu-link" H 1008 5290 50  0000 C CNN
-F 2 "Connector_PinSocket_2.54mm:PinSocket_1x05_P2.54mm_Vertical" H 900 5000 50  0001 C CNN
-F 3 "~" H 900 5000 50  0001 C CNN
-	1    900  5000
-	1    0    0    -1
+P 1400 5050
+F 0 "J3" H 1508 5431 50  0000 C CNN
+F 1 "Nu-link" H 1508 5340 50  0000 C CNN
+F 2 "Connector_PinSocket_2.54mm:PinSocket_1x05_P2.54mm_Vertical" H 1400 5050 50  0001 C CNN
+F 3 "~" H 1400 5050 50  0001 C CNN
+	1    1400 5050
+	-1   0    0    1
 $EndComp
 $Comp
 L power:VDD #PWR0110
 U 1 1 5F0A501C
-P 1300 4800
-F 0 "#PWR0110" H 1300 4650 50  0001 C CNN
-F 1 "VDD" V 1317 4928 50  0000 L CNN
-F 2 "" H 1300 4800 50  0001 C CNN
-F 3 "" H 1300 4800 50  0001 C CNN
-	1    1300 4800
-	0    1    1    0
+P 1000 4850
+F 0 "#PWR0110" H 1000 4700 50  0001 C CNN
+F 1 "VDD" V 1017 4978 50  0000 L CNN
+F 2 "" H 1000 4850 50  0001 C CNN
+F 3 "" H 1000 4850 50  0001 C CNN
+	1    1000 4850
+	1    0    0    -1
 $EndComp
 $Comp
 L power:GND #PWR0111
 U 1 1 5F0A57BB
-P 1300 5250
-F 0 "#PWR0111" H 1300 5000 50  0001 C CNN
-F 1 "GND" H 1305 5077 50  0000 C CNN
-F 2 "" H 1300 5250 50  0001 C CNN
-F 3 "" H 1300 5250 50  0001 C CNN
-	1    1300 5250
-	1    0    0    -1
-$EndComp
-Wire Wire Line
-	1100 5200 1300 5200
-Wire Wire Line
-	1300 5200 1300 5250
-Wire Wire Line
-	1100 4800 1300 4800
+P 1000 5250
+F 0 "#PWR0111" H 1000 5000 50  0001 C CNN
+F 1 "GND" H 1005 5077 50  0000 C CNN
+F 2 "" H 1000 5250 50  0001 C CNN
+F 3 "" H 1000 5250 50  0001 C CNN
+	1    1000 5250
+	1    0    0    -1
+$EndComp
+Wire Wire Line
+	1200 4850 1000 4850
+Wire Wire Line
+	1200 5250 1000 5250
 Text Label 5400 4750 0    50   ~ 0
 DCK
@@
 DDA
 Wire Wire Line
-	1100 4900 1300 4900
-Wire Wire Line
-	1100 5000 1300 5000
-Wire Wire Line
-	1100 5100 1300 5100
-Text Label 1300 4900 0    50   ~ 0
+	1200 5150 1000 5150
+Wire Wire Line
+	1200 5050 1000 5050
+Wire Wire Line
+	1200 4950 1000 4950
+Text Label 1000 4950 2    50   ~ 0
 DDA
-Text Label 1300 5000 0    50   ~ 0
+Text Label 1000 5050 2    50   ~ 0
 DCK
-Text Label 1300 5100 0    50   ~ 0
+Text Label 1000 5150 2    50   ~ 0
 RST
 $Comp
