File: hard/_autosave-XS40.sch (KiCad schematic (older format))
At the start: 94 parts, among them J1 USB_B_Micro, J2 Conn_01x20_Female, J3 Nu-link, SW1 SW_Push, SW10 SW_Push, SW11 SW_Push, SW12 SW_Push, SW13 SW_Push, SW14 SW_Push, SW15 SW_Push, SW16 SW_Push, SW17 SW_Push, SW18 SW_Push, SW19 SW_Push, SW2 SW_Push, SW20 SW_Push, SW21 SW_Push, SW22 SW_Push, SW23 SW_Push, SW24 SW_Push, SW25 SW_Push, SW26 SW_Push, SW27 SW_Push, SW28 SW_Push, SW29 SW_Push, SW3 SW_Push, SW30 SW_Push, SW31 SW_Push, SW32 SW_Push, SW33 SW_Push, SW34 SW_Push, SW35 SW_Push, SW36 SW_Push, SW37 SW_Push, SW38 SW_Push, SW39 SW_Push, SW4 SW_Push, SW40 SW_Push, SW5 SW_Push, SW6 SW_Push, SW7 SW_Push, SW8 SW_Push, SW9 SW_Push, U1 N76E003AT20, U2 CH9328

Commit message: PCB添加了少的一根GND线，打包存档v0.1
Parts:
- added P44: USB_C_Plug, symbol Connector:USB_C_Plug
Changed lines of the file:
@@
 Wire Wire Line
 	1900 5150 1900 4850
+$Comp
+L Connector:USB_C_Plug P44
+U 1 1 5E7A39F3
+P 6750 5100
+F 0 "P44" H 6857 6367 50  0000 C CNN
+F 1 "USB_C_Plug" H 6857 6276 50  0000 C CNN
+F 2 "" H 6900 5100 50  0001 C CNN
+F 3 "https://www.usb.org/sites/default/files/documents/usb_type-c.zip" H 6900 5100 50  0001 C CNN
+	1    6750 5100
+	1    0    0    -1
+$EndComp
 $EndSCHEMATC
